File: Linear Power Supply.kicad_pcb (KiCad board)
At the start: 2 copper layers, 9 parts, among them SW1 SW_Nidec_CAS-120A1, U1 L7805

Commit message: fix issue
Parts:
- added R2: 2K, Resistor_THT:R_Axial_DIN0204_L3.6mm_D1.6mm_P5.08mm_Horizontal, F.Cu at (122.9, 103.9)
- added R3: 2K, Resistor_THT:R_Axial_DIN0204_L3.6mm_D1.6mm_P5.08mm_Horizontal, F.Cu at (132.3, 104.4)
- R1: value 100K -> 100
- moved U1 22.2 mm to (168.1, 77.5)
- moved R1 20.9 mm to (92.7, 63.0)
- moved D1 20.7 mm to (85.9, 54.6)
- moved D2 5.52 mm to (140.8, 82.7)
Connections:
- D2 pad 2: unconnected-(SW1-A-Pad3) -> Net-(SW1-B)
- D2 pad 3: Net-(SW1-B) -> unconnected-(D2-AC-Pad3)
Routing:
- net Net-(D2-VCC): track 128.0 -> 171.5 mm
- net Net-(U1-OUT): track 70.7 -> 110.2 mm
- net GND: track 217.7 -> 246.8 mm
- net unconnected-(L1-OUT+-Pad7): track 9.53 -> 0.00 mm, vias 1 -> 0
- net (no net): track 20.7 -> 30.0 mm, vias 1 -> 2
- net unconnected-(SW1-A-Pad3): track 14.3 -> 20.2 mm
- net unconnected-(SW1-C-Pad1): track 6.04 -> 9.61 mm
- net Net-(SW1-B): track 8.28 -> 10.5 mm
